Commit message: real uf850 + xarm gripper meshes, full-screen dashboard
phase 15-20 (post-audit pass):
- audited urdf against ufactory 850 datasheet — joint ranges, speeds,
  torques, reach all match official spec.
- stripped the fake table; props sit on bare floor.
- added robot mount pedestal (205 mm, part of every real uf850
  installation, not a 'table'). visible cylinder in renders.
- swapped the hand-rolled parallel jaw for the real xarm gripper:
  base_link.stl + left/right outer knuckle + finger + inner knuckle
  meshes from xarm_ros2, 4-bar linkage with 5 mimic joints expressed
  via mujoco equality constraints. tcp at 172 mm from flange per
  the xarm gripper datasheet.
- collision groups (contype/conaffinity) so the gripper fingers can
  pass close to the floor without destabilizing contact when reaching
  for low props; props collide with floor + arm + each other.
- two-stage axis-only ik (position then axis alignment), gripper-down
  with free yaw — opens up the floor-level workspace the wrist limit
  otherwise blocks.
- full-screen dashboard: home page is 3d viewer + right rail, run
  detail page is viewer + live event timeline. arm fills the screen.
verification: 244 + 21 + 51 + 3 = 319 tests green. all linters clean.
5 freeform llm-decomposed tasks executed end-to-end via the dashboard,
including a 2-step decomposition ('make a tower with all three
blocks' → stack red on blue, stack green on red).

File: farm-cloud/ui/public/urdf/uf850/uf850.urdf (robot description, URDF)
Before this commit: robot uf850, 12 links, 11 joints
Links:
- removed link finger_left
- removed link finger_right
- removed link gripper_base
- removed link link_eef
- added link left_finger, mass 0.048304; visual mesh filename=meshes/gripper/left_finger.stl
- added link left_inner_knuckle, mass 0.023013; visual mesh filename=meshes/gripper/left_inner_knuckle.stl
- added link left_outer_knuckle, mass 0.033618; visual mesh filename=meshes/gripper/left_outer_knuckle.stl
- added link mount; visual cylinder length=0.01 radius=0.10; visual cylinder length=0.01 radius=0.12
- added link right_finger, mass 0.048304; visual mesh filename=meshes/gripper/right_finger.stl
- added link right_inner_knuckle, mass 0.023013; visual mesh filename=meshes/gripper/right_inner_knuckle.stl
- added link right_outer_knuckle, mass 0.033618; visual mesh filename=meshes/gripper/right_outer_knuckle.stl
- added link world
- added link xarm_gripper_base_link, mass 0.54156; visual mesh filename=meshes/gripper/base_link.stl
- link link1: geometry visual mesh filename=meshes/visual/link1.stl
- link link2: geometry visual mesh filename=meshes/visual/link2.stl
- link link3: geometry visual mesh filename=meshes/visual/link3.stl
- link link4: geometry visual mesh filename=meshes/visual/link4.stl
- link link5: geometry visual mesh filename=meshes/visual/link5.stl
- link link6: geometry visual mesh filename=meshes/visual/link6.stl
- link link_base: geometry visual mesh filename=meshes/visual/link_base.stl
Joints:
- removed joint finger_left_joint
- removed joint finger_right_joint
- removed joint joint_eef
- removed joint joint_gripper_base
- added joint drive_joint: type revolute, parent xarm_gripper_base_link, child left_outer_knuckle, origin xyz=0 0.035 0.059098 rpy=0 0 0, axis 1 0 0, limit lower=0 upper=0.85 effort=50 velocity=2
- added joint left_finger_joint: type revolute, parent left_outer_knuckle, child left_finger, origin xyz=0 0.035465 0.042039 rpy=0 0 0, axis -1 0 0, limit lower=0 upper=0.85 effort=50 velocity=2, mimic joint=drive_joint multiplier=1 offset=0
- added joint left_inner_knuckle_joint: type revolute, parent xarm_gripper_base_link, child left_inner_knuckle, origin xyz=0 0.02 0.074098 rpy=0 0 0, axis 1 0 0, limit lower=0 upper=0.85 effort=50 velocity=2, mimic joint=drive_joint multiplier=1 offset=0
- added joint link_base_to_mount: type fixed, parent mount, child link_base, origin xyz=0 0 0.205
- added joint mount_to_world: type fixed, parent world, child mount, origin xyz=0 0 0
- added joint right_finger_joint: type revolute, parent right_outer_knuckle, child right_finger, origin xyz=0 -0.035465 0.042039 rpy=0 0 0, axis 1 0 0, limit lower=0 upper=0.85 effort=50 velocity=2, mimic joint=drive_joint multiplier=1 offset=0
- added joint right_inner_knuckle_joint: type revolute, parent xarm_gripper_base_link, child right_inner_knuckle, origin xyz=0 -0.02 0.074098 rpy=0 0 0, axis -1 0 0, limit lower=0 upper=0.85 effort=50 velocity=2, mimic joint=drive_joint multiplier=1 offset=0
- added joint right_outer_knuckle_joint: type revolute, parent xarm_gripper_base_link, child right_outer_knuckle, origin xyz=0 -0.035 0.059098 rpy=0 0 0, axis -1 0 0, limit lower=0 upper=0.85 effort=50 velocity=2, mimic joint=drive_joint multiplier=1 offset=0
- added joint xarm_gripper_fix: type fixed, parent link6, child xarm_gripper_base_link, origin xyz=0 0 0
- joint joint_tcp: origin xyz=0 0 0.08 rpy=0 0 0 -> xyz=0 0 0.172 rpy=0 0 0; parent gripper_base -> xarm_gripper_base_link

Commit message: fix arm/block sync + pi0.5 inference scaffold
arm/block sync (#23):
- root cause: mjcf default eulerseq is *intrinsic* xyz, urdf rpy is
  *extrinsic* xyz. same rpy values in both files produced different
  joint frames (offsets at joints 2 and 3 are particularly affected).
  the mjcf simulated one robot, the urdf-loader viewer rendered a
  *different* robot at the same joint values — so blocks moved
  correctly (sim is ground truth) but the arm in the dashboard
  appeared misaligned.
- fix: converted mjcf intrinsic rpy for joints 2 and 3 to their
  extrinsic-xyz equivalents in the urdf. urdf forward kinematics now
  agrees with mjcf to 0.0 mm at the tcp site. also rebuilt the urdf
  gripper as the same simple 2-slider + mimic as the mjcf so finger
  motion matches.
pi0.5 vla model (#22):
- added 2 cameras to mjcf (exterior + wrist, mode='targetbody').
- simdriver.pi05_observation() returns the droid-policy dict shape
  (224×224 uint8 images, 7-dim joint state, 1-dim gripper).
- simdriver.apply_joint_action() executes joint deltas + gripper
  target at the model's control rate.
- new policies/pi05.py: http client for the modal-hosted endpoint
  plus the closed-loop runner that calls infer → step n actions →
  observe → repeat.
- new farm-cloud/modal/pi05_serve.py: deployable modal app that
  loads pi05_droid on an a100 and exposes /infer.
- supervisor branches to the pi0.5 path when FARM_POLICY=pi05 or
  FARM_PI05_ENDPOINT is configured; falls back to gpt skills
  otherwise. all events route through the run record + sse bus.

File: farm-cloud/ui/public/urdf/uf850/uf850.urdf (robot description, URDF)
Before this commit: robot uf850, 17 links, 16 joints
Links:
- removed link left_inner_knuckle
- removed link left_outer_knuckle
- removed link right_inner_knuckle
- removed link right_outer_knuckle
- link left_finger: mass 0.048304 -> 0.05
- link right_finger: mass 0.048304 -> 0.05
- link xarm_gripper_base_link: geometry visual mesh filename=meshes/gripper/base_link.stl; visual mesh filename=meshes/gripper/left_inner_knuckle.stl
Joints:
- removed joint drive_joint
- removed joint left_inner_knuckle_joint
- removed joint right_inner_knuckle_joint
- removed joint right_outer_knuckle_joint
- joint joint2: origin xyz=0 0 0 rpy=1.5708 -1.5708 0 -> xyz=0 0 0 rpy=1.5708 0 -1.5708
- joint joint3: origin xyz=0.39 0 0 rpy=-3.1416 0 -1.5708 -> xyz=0.39 0 0 rpy=-3.1416 0 1.5708
- joint left_finger_joint: axis -1 0 0 -> 0 -1 0; limit lower=0 upper=0.85 effort=50 velocity=2 -> lower=0 upper=0.035 effort=50 velocity=0.5; mimic joint=drive_joint multiplier=1 offset=0 -> (none); origin xyz=0 0.035465 0.042039 rpy=0 0 0 -> xyz=0 0.035 0.100 rpy=0 0 0; parent left_outer_knuckle -> xarm_gripper_base_link; type revolute -> prismatic
- joint right_finger_joint: axis 1 0 0 -> 0 1 0; limit lower=0 upper=0.85 effort=50 velocity=2 -> lower=0 upper=0.035 effort=50 velocity=0.5; mimic joint=drive_joint multiplier=1 offset=0 -> joint=left_finger_joint multiplier=1 offset=0; origin xyz=0 -0.035465 0.042039 rpy=0 0 0 -> xyz=0 -0.035 0.100 rpy=0 0 0; parent right_outer_knuckle -> xarm_gripper_base_link; type revolute -> prismatic
