Commit message: digital Setup

File: farm-edge-agent/assets/urdf/uf850/uf850.urdf (robot description, URDF)
Before this commit: robot uf850, 13 links, 12 joints
Links:
- removed link mount
- removed link tcp
- added link left_inner_knuckle, mass 0.0230125781256706; collision mesh filename=meshes/gripper/left_inner_knuckle.stl; visual mesh filename=meshes/gripper/left_inner_knuckle.stl
- added link left_outer_knuckle, mass 0.033618; collision mesh filename=meshes/gripper/left_outer_knuckle.stl; visual mesh filename=meshes/gripper/left_outer_knuckle.stl
- added link link_eef
- added link link_tcp
- added link right_inner_knuckle, mass 0.023013; collision mesh filename=meshes/gripper/right_inner_knuckle.stl; visual mesh filename=meshes/gripper/right_inner_knuckle.stl
- added link right_outer_knuckle, mass 0.033618; collision mesh filename=meshes/gripper/right_outer_knuckle.stl; visual mesh filename=meshes/gripper/right_outer_knuckle.stl
- link left_finger: mass 0.05 -> 0.048304; geometry collision mesh filename=meshes/gripper/left_finger.stl; visual mesh filename=meshes/gripper/left_finger.stl
- link link1: mass 2.16 -> 4.807; geometry collision mesh filename=meshes/collision/link1.stl; visual mesh filename=meshes/visual/link1.stl
- link link2: mass 2.04 -> 3.28; geometry collision mesh filename=meshes/collision/link2.stl; visual mesh filename=meshes/visual/link2.stl
- link link3: mass 1.7 -> 2.237; geometry collision mesh filename=meshes/collision/link3.stl; visual mesh filename=meshes/visual/link3.stl
- link link4: mass 1.34 -> 2.041; geometry collision mesh filename=meshes/collision/link4.stl; visual mesh filename=meshes/visual/link4.stl
- link link5: mass 1.16 -> 1.385; geometry collision mesh filename=meshes/collision/link5.stl; visual mesh filename=meshes/visual/link5.stl
- link link6: mass 0.17 -> 0.225; geometry collision mesh filename=meshes/collision/link6.stl; visual mesh filename=meshes/visual/link6.stl
- link link_base: geometry collision mesh filename=meshes/collision/link_base.stl; visual mesh filename=meshes/visual/link_base.stl
- link right_finger: mass 0.05 -> 0.048304; geometry collision mesh filename=meshes/gripper/right_finger.stl; visual mesh filename=meshes/gripper/right_finger.stl
- link xarm_gripper_base_link: geometry collision mesh filename=meshes/gripper/base_link.stl; visual mesh filename=meshes/gripper/base_link.stl
Joints:
- removed joint link_base_to_mount
- removed joint mount_to_world
- removed joint xarm_gripper_fix
- added joint drive_joint: type revolute, parent xarm_gripper_base_link, child left_outer_knuckle, origin xyz=0 0.035 0.059098 rpy=0 0 0, axis 1 0 0, limit lower=0 upper=0.85 effort=50 velocity=2
- added joint gripper_fix: type fixed, parent link_eef, child xarm_gripper_base_link, origin xyz=0 0 0 rpy=0 0 0
- added joint joint_eef: type fixed, parent link6, child link_eef, origin xyz=0 0 0 rpy=0 0 0
- added joint left_inner_knuckle_joint: type revolute, parent xarm_gripper_base_link, child left_inner_knuckle, origin xyz=0 0.02 0.074098 rpy=0 0 0, axis 1 0 0, limit lower=0 upper=0.85 effort=50 velocity=2, mimic joint=drive_joint multiplier=1 offset=0
- added joint right_inner_knuckle_joint: type revolute, parent xarm_gripper_base_link, child right_inner_knuckle, origin xyz=0 -0.02 0.074098 rpy=0 0 0, axis -1 0 0, limit lower=0 upper=0.85 effort=50 velocity=2, mimic joint=drive_joint multiplier=1 offset=0
- added joint right_outer_knuckle_joint: type revolute, parent xarm_gripper_base_link, child right_outer_knuckle, origin xyz=0 -0.035 0.059098 rpy=0 0 0, axis -1 0 0, limit lower=0 upper=0.85 effort=50 velocity=2, mimic joint=drive_joint multiplier=1 offset=0
- added joint world_joint: type fixed, parent world, child link_base, origin xyz=0 0 0 rpy=0 0 0
- joint joint1: limit lower=-6.283185 upper=6.283185 effort=200 velocity=3.14 -> lower=-6.283185307179586 upper=6.283185307179586 effort=200.0 velocity=3.14
- joint joint2: limit lower=-2.3038346 upper=2.3038346 effort=200 velocity=3.14 -> lower=-2.3038346 upper=2.3038346 effort=200.0 velocity=3.14; origin xyz=0 0 0 rpy=1.5708 0 -1.5708 -> xyz=0 0 0 rpy=1.5708 -1.5708 0
- joint joint3: limit lower=-4.2236968 upper=0.061087 effort=90 velocity=3.14 -> lower=-4.2236968 upper=0.061087 effort=90.0 velocity=3.14; origin xyz=0.39 0 0 rpy=-3.1416 0 1.5708 -> xyz=0.39 0 0 rpy=-3.1416 0 -1.5708
- joint joint4: limit lower=-6.283185 upper=6.283185 effort=68 velocity=3.14 -> lower=-6.283185307179586 upper=6.283185307179586 effort=68.0 velocity=3.14
- joint joint5: limit lower=-2.1642 upper=2.1642 effort=19 velocity=3.14 -> lower=-2.1642 upper=2.1642 effort=19.0 velocity=3.14
- joint joint6: limit lower=-6.283185 upper=6.283185 effort=19 velocity=3.14 -> lower=-6.283185307179586 upper=6.283185307179586 effort=19.0 velocity=3.14
- joint joint_tcp: child tcp -> link_tcp
- joint left_finger_joint: axis 0 -1 0 -> -1 0 0; limit lower=0 upper=0.035 effort=50 velocity=0.5 -> lower=0 upper=0.85 effort=50 velocity=2; mimic (none) -> joint=drive_joint multiplier=1 offset=0; origin xyz=0 0.035 0.100 rpy=0 0 0 -> xyz=0 0.035465 0.042039 rpy=0 0 0; parent xarm_gripper_base_link -> left_outer_knuckle; type prismatic -> revolute
- joint right_finger_joint: axis 0 1 0 -> 1 0 0; limit lower=0 upper=0.035 effort=50 velocity=0.5 -> lower=0 upper=0.85 effort=50 velocity=2; mimic joint=left_finger_joint multiplier=1 offset=0 -> joint=drive_joint multiplier=1 offset=0; origin xyz=0 -0.035 0.100 rpy=0 0 0 -> xyz=0 -0.035465 0.042039 rpy=0 0 0; parent xarm_gripper_base_link -> right_outer_knuckle; type prismatic -> revolute
